Commit message: use larger indentation for readability

File: urdf/arm.xacro (robot description, xacro)
@@ -1,40 +1,38 @@
 <?xml version="1.0"?>
 <robot xmlns:xacro="http://www.ros.org/wiki/xacro" name="my_robot">
-  <xacro:macro name="arm" params="prefix radius length reflect">
+<xacro:macro name="arm" params="prefix radius length reflect">
     <link name="${prefix}_arm">
-      <visual>
-        <origin rpy="0 0 0" xyz="0 0 0.04"/>
-        <geometry>
-          <cylinder length="${length}" radius="${radius}"/>
-        </geometry>
-        <material name="my_colour">
-          <color rgba="0 1.0 1.0 0"/>
-        </material>
-      </visual>
-      <collision>
-        <geometry>
-          <cylinder length="${length}" radius="${radius}"/>
-        </geometry>
-      </collision>
-      <inertial>
-        <mass value="1"/>
-        <inertia ixx="0.06" ixy="0.0" ixz="0.0" iyy="0.06" iyz="0.0" izz="0.25"/>
-      </inertial>
+        <visual>
+            <origin rpy="0 0 0" xyz="0 0 0.04"/>
+            <geometry>
+                <cylinder length="${length}" radius="${radius}"/>
+            </geometry>
+        </visual>
+        <collision>
+            <geometry>
+                <cylinder length="${length}" radius="${radius}"/>
+            </geometry>
+        </collision>
+        <inertial>
+            <mass value="1"/>
+            <inertia ixx="0.06" ixy="0.0" ixz="0.0" iyy="0.06" iyz="0.0" izz="0.25"/>
+        </inertial>
     </link>
     <joint name="base_to_${prefix}_arm" type="continuous">
-      <axis xyz="0 1 0"/>
-      <parent link="base_link"/>
-      <child link="${prefix}_arm"/>
-      <origin rpy="0 0 0" xyz="0 ${0.06*reflect} 0.0"/>
+        <axis xyz="0 1 0"/>
+        <parent link="base_link"/>
+        <child link="${prefix}_arm"/>
+        <origin rpy="0 0 0" xyz="0 ${0.06*reflect} 0.0"/>
+        <limit effort="30" velocity="1.0"/>
     </joint>
     <transmission name="${prefix}_arm_transmission">
-      <type>transmission_interface/SimpleTransmission</type>
-      <actuator name="$${prefix}_motor">
-        <mechanicalReduction>1</mechanicalReduction>
-      </actuator>
-      <joint name="base_to_${prefix}_arm">
-        <hardwareInterface>hardware_interface/VelocityJointInterface</hardwareInterface>
-      </joint>
+        <type>transmission_interface/SimpleTransmission</type>
+        <actuator name="$${prefix}_motor">
+            <mechanicalReduction>1</mechanicalReduction>
+        </actuator>
+        <joint name="base_to_${prefix}_arm">
+            <hardwareInterface>hardware_interface/VelocityJointInterface</hardwareInterface>
+        </joint>
     </transmission>
-  </xacro:macro>
+</xacro:macro>
 </robot>

File: urdf/bot.xacro (robot description, xacro)
@@ -1,30 +1,30 @@
 <?xml version="1.0"?>
 <robot xmlns:xacro="http://www.ros.org/wiki/xacro" name="my_robot">
-  <xacro:include filename="$(find tutorial)/urdf/arm.xacro" />
-  <xacro:include filename="$(find tutorial)/urdf/head.xacro" />
-  <link name="base_link">
-    <visual>
-      <geometry>
-        <box size=".07 .09 .12"/>
-      </geometry>
-    </visual>
-    <collision>
-      <geometry>
-        <box size=".07 .09 .12"/>
-      </geometry>
-    </collision>
-    <inertial>
-      <mass value="1"/>
-      <inertia ixx="0.21" ixy="0.00" ixz="0.00" iyy="0.27" iyz="0.00" izz="0.10"/>
-    </inertial>
-  </link>
-  <xacro:arm prefix="right" length="0.06" radius="0.01" reflect="1" />
-  <xacro:arm prefix="left" length="0.06" radius="0.01" reflect="-1" />
-  <xacro:head />
-  <!-- Add ROS plugin so we can interact with our robot -->
-  <gazebo>
-    <plugin name="gazebo_ros_control" filename="libgazebo_ros_control.so">
-      <robotNamespace>/</robotNamespace>
-    </plugin>
-  </gazebo>
+    <xacro:include filename="$(find tutorial)/urdf/arm.xacro" />
+    <xacro:include filename="$(find tutorial)/urdf/head.xacro" />
+    <link name="base_link">
+        <visual>
+            <geometry>
+                <box size=".07 .09 .12"/>
+            </geometry>
+        </visual>
+        <collision>
+            <geometry>
+                <box size=".07 .09 .12"/>
+            </geometry>
+        </collision>
+        <inertial>
+            <mass value="1"/>
+            <inertia ixx="0.21" ixy="0.00" ixz="0.00" iyy="0.27" iyz="0.00" izz="0.10"/>
+        </inertial>
+    </link>
+    <xacro:arm prefix="right" length="0.06" radius="0.01" reflect="1" />
+    <xacro:arm prefix="left" length="0.06" radius="0.01" reflect="-1" />
+    <xacro:head />
+    <!-- Add ROS plugin so we can interact with our robot -->
+    <gazebo>
+        <plugin name="gazebo_ros_control" filename="libgazebo_ros_control.so">
+            <robotNamespace>/</robotNamespace>
+        </plugin>
+    </gazebo>
 </robot>

File: urdf/head.xacro (robot description, xacro)
@@ -1,37 +1,37 @@
 <?xml version="1.0"?>
 <robot xmlns:xacro="http://www.ros.org/wiki/xacro" name="my_robot">
-  <xacro:macro name="head">
+<xacro:macro name="head">
     <link name="head_link">
-      <visual>
-        <geometry>
-          <mesh filename="package://tutorial/urdf/head.dae" scale=".5 .5 .5"/>
-        </geometry>
-      </visual>
-      <collision>
-        <geometry>
-          <sphere radius="0.02"/>
-        </geometry>
-      </collision>
-      <inertial>
-        <mass value="0.10"/>
-        <inertia ixx="0.03" ixy="0.0" ixz="0.0" iyy="0.03" iyz="0.0" izz="0.03"/>
-      </inertial>
+        <visual>
+            <geometry>
+                <mesh filename="package://tutorial/urdf/head.dae" scale=".5 .5 .5"/>
+            </geometry>
+        </visual>
+        <collision>
+            <geometry>
+                <sphere radius="0.02"/>
+            </geometry>
+        </collision>
+        <inertial>
+            <mass value="0.10"/>
+            <inertia ixx="0.03" ixy="0.0" ixz="0.0" iyy="0.03" iyz="0.0" izz="0.03"/>
+        </inertial>
     </link>
     <joint name="base_to_head" type="continuous">
-      <axis xyz="0 0 1"/>
-      <parent link="base_link"/>
-      <child link="head_link"/>
-      <origin rpy="0 0 0" xyz="0 0 0.05"/>
-      <limit effort="30" velocity="1.0"/>
+        <axis xyz="0 0 1"/>
+        <parent link="base_link"/>
+        <child link="head_link"/>
+        <origin rpy="0 0 0" xyz="0 0 0.05"/>
+        <limit effort="30" velocity="1.0"/>
     </joint>
     <transmission name="head_transmission">
-      <type>transmission_interface/SimpleTransmission</type>
-      <actuator name="$head_motor">
-        <mechanicalReduction>1</mechanicalReduction>
-      </actuator>
-      <joint name="base_to_head">
-        <hardwareInterface>hardware_interface/PositionJointInterface</hardwareInterface>
-      </joint>
+        <type>transmission_interface/SimpleTransmission</type>
+        <actuator name="$head_motor">
+            <mechanicalReduction>1</mechanicalReduction>
+        </actuator>
+        <joint name="base_to_head">
+            <hardwareInterface>hardware_interface/PositionJointInterface</hardwareInterface>
+        </joint>
     </transmission>
-  </xacro:macro>
+</xacro:macro>
 </robot>

Commit message: simplify values and add helpful comments

File: urdf/arm.xacro (robot description, xacro)
@@ -2,7 +2,9 @@
 <robot xmlns:xacro="http://www.ros.org/wiki/xacro" name="my_robot">
 <xacro:macro name="arm" params="prefix radius length reflect">
+    <!-- rpy (roll pitch yaw) describes rotation in radians -->
+    <!-- xyz describes translation in meters -->
     <link name="${prefix}_arm">
         <visual>
-            <origin rpy="0 0 0" xyz="0 0 0.04"/>
+            <origin rpy="0 0 0" xyz="0 0 1"/> <!-- set the origin to 0 to recenter the link to the child_frame -->
             <geometry>
                 <cylinder length="${length}" radius="${radius}"/>
@@ -10,4 +12,5 @@
         </visual>
         <collision>
+            <origin rpy="0 0 0" xyz="0 0 1"/> <!-- set the origin to 0 to recenter the link to the child_frame -->
             <geometry>
                 <cylinder length="${length}" radius="${radius}"/>
@@ -15,4 +18,5 @@
         </collision>
         <inertial>
+            <origin rpy="0 0 0" xyz="0 0 1"/> <!-- set the origin to 0 to recenter the link to the child_frame -->
             <mass value="1"/>
             <inertia ixx="0.06" ixy="0.0" ixz="0.0" iyy="0.06" iyz="0.0" izz="0.25"/>
@@ -23,5 +27,5 @@
         <parent link="base_link"/>
         <child link="${prefix}_arm"/>
-        <origin rpy="0 0 0" xyz="0 ${0.06*reflect} 0.0"/>
+        <origin rpy="0.2 0 0" xyz="0 ${reflect*0.7} 0"/> <!-- move the child_frame with respect to parent_frame -->
         <limit effort="30" velocity="1.0"/>
     </joint>

File: urdf/head.xacro (robot description, xacro)
@@ -4,23 +4,26 @@
     <link name="head_link">
         <visual>
+            <origin rpy="0 0 0" xyz="0 0 0"/>
             <geometry>
-                <mesh filename="package://tutorial/urdf/head.dae" scale=".5 .5 .5"/>
+                <mesh filename="package://tutorial/urdf/head.dae" scale="5 5 5"/>
             </geometry>
         </visual>
         <collision>
+            <origin rpy="0 0 0" xyz="0 0 0"/>
             <geometry>
-                <sphere radius="0.02"/>
+                <sphere radius=".2"/>
             </geometry>
         </collision>
         <inertial>
-            <mass value="0.10"/>
+            <origin rpy="0 0 0" xyz="0 0 0"/>
+            <mass value="1"/>
             <inertia ixx="0.03" ixy="0.0" ixz="0.0" iyy="0.03" iyz="0.0" izz="0.03"/>
         </inertial>
     </link>
     <joint name="base_to_head" type="continuous">
-        <axis xyz="0 0 1"/>
+        <axis xyz="0 0 1"/>  <!-- changes axis of rotation -->
         <parent link="base_link"/>
         <child link="head_link"/>
-        <origin rpy="0 0 0" xyz="0 0 0.05"/>
+        <origin rpy="0 0 0" xyz="0 0 .5"/> <!-- moves the child_frame with respect to parent_frame -->
         <limit effort="30" velocity="1.0"/>
     </joint>

File: urdf/main.xacro (robot description, xacro)
@@ -6,19 +6,19 @@
         <visual>
             <geometry>
-                <box size=".07 .09 .12"/>
+                <box size="1 1 1"/>
             </geometry>
         </visual>
         <collision>
             <geometry>
-                <box size=".07 .09 .12"/>
+                <box size="1 1 1"/>
             </geometry>
         </collision>
         <inertial>
             <mass value="1"/>
-            <inertia ixx="0.21" ixy="0.00" ixz="0.00" iyy="0.27" iyz="0.00" izz="0.10"/>
+            <inertia ixx="0.21" ixy="0" ixz="0" iyy="0.27" iyz="0" izz="0.10"/>
         </inertial>
     </link>
-    <xacro:arm prefix="right" length="0.06" radius="0.01" reflect="1" />
-    <xacro:arm prefix="left" length="0.06" radius="0.01" reflect="-1" />
+    <xacro:arm prefix="right" length=".7" radius=".2" reflect="1" />
+    <xacro:arm prefix="left" length=".7" radius=".2" reflect="-1" />
     <xacro:head />
     <!-- Add ROS plugin so we can interact with our robot -->

Commit message: i did stuff i did a lot of work

File: urdf/arm.xacro (robot description, xacro)
@@ -1,22 +1,22 @@
 <?xml version="1.0"?>
 <robot xmlns:xacro="http://www.ros.org/wiki/xacro" name="my_robot">
-<xacro:macro name="arm" params="prefix radius length reflect">
+<xacro:macro name="arm" params="prefix radius length reflect_x reflect_y">
     <!-- rpy (roll pitch yaw) describes rotation in radians -->
     <!-- xyz describes translation in meters -->
     <link name="${prefix}_arm">
         <visual>
-            <origin rpy="0 0 0" xyz="0 0 1"/> <!-- set the origin to 0 to recenter the link to the child_frame -->
+            <origin rpy="${pi/2} 0 0" xyz="0 0 0"/> <!-- set the origin to 0 to recenter the link to the child_frame -->
             <geometry>
-                <cylinder length="${length}" radius="${radius}"/>
+            	<cylinder length="${length}" radius="${radius}"/>
             </geometry>
         </visual>
         <collision>
-            <origin rpy="0 0 0" xyz="0 0 1"/> <!-- set the origin to 0 to recenter the link to the child_frame -->
+            <origin rpy="${pi/2} 0 0" xyz="0 0 0"/> <!-- set the origin to 0 to recenter the link to the child_frame -->
             <geometry>
-                <cylinder length="${length}" radius="${radius}"/>
+             	<cylinder length="${length}" radius="${radius}"/>
             </geometry>
         </collision>
         <inertial>
-            <origin rpy="0 0 0" xyz="0 0 1"/> <!-- set the origin to 0 to recenter the link to the child_frame -->
+            <origin rpy="${pi/2} 0 0" xyz="0 0 0"/> <!-- set the origin to 0 to recenter the link to the child_frame -->
             <mass value="1"/>
             <inertia ixx="0.06" ixy="0.0" ixz="0.0" iyy="0.06" iyz="0.0" izz="0.25"/>
@@ -25,8 +25,29 @@
     <joint name="base_to_${prefix}_arm" type="continuous">
         <axis xyz="0 1 0"/>
+        <parent link="${prefix}_arm_turn"/>
+        <child link="${prefix}_arm"/>
+        <origin rpy="0 0 0" xyz="0 0 0"/> <!-- move the child_frame with respect to parent_frame -->
+        <limit effort="30" velocity="5.0"/>
+    </joint>
+ <link name="${prefix}_arm_turn">
+	<visual>
+            <origin rpy="0 0 0" xyz="0 0 0"/> <!-- set the origin to 0 to recenter the link to the child_frame -->
+            <geometry>
+            </geometry>
+        </visual>
+        <collision>
+        </collision>
+        <inertial>
+            <origin rpy="${pi/2} 0 0" xyz="0 0 0"/> <!-- set the origin to 0 to recenter the link to the child_frame -->
+            <mass value="1"/>
+            <inertia ixx="0.06" ixy="0.0" ixz="0.0" iyy="0.06" iyz="0.0" izz="0.25"/>
+        </inertial>
+    </link>
+    <joint name="base_to_${prefix}_arm_turn" type="continuous">
+        <axis xyz="0 0 1"/>
         <parent link="base_link"/>
-        <child link="${prefix}_arm"/>
-        <origin rpy="0.2 0 0" xyz="0 ${reflect*0.7} 0"/> <!-- move the child_frame with respect to parent_frame -->
-        <limit effort="30" velocity="1.0"/>
+        <child link="${prefix}_arm_turn"/>
+        <origin rpy="0 0 0" xyz="${reflect_x*0.6} ${reflect_y*0.6} 0"/> <!-- move the child_frame with respect to parent_frame -->
+        <limit effort="30" velocity="5.0"/>
     </joint>
     <transmission name="${prefix}_arm_transmission">
@@ -39,4 +60,13 @@
         </joint>
     </transmission>
+    <transmission name="${prefix}_arm_transmission_turn">
+        <type>transmission_interface/SimpleTransmission</type>
+        <actuator name="$${prefix}_motor">
+            <mechanicalReduction>1</mechanicalReduction>
+        </actuator>
+        <joint name="base_to_${prefix}_arm_turn">
+            <hardwareInterface>hardware_interface/PositionJointInterface</hardwareInterface>
+        </joint>
+    </transmission>
 </xacro:macro>
 </robot>

File: urdf/head.xacro (robot description, xacro)
@@ -4,5 +4,5 @@
     <link name="head_link">
         <visual>
-            <origin rpy="0 0 0" xyz="0 0 0"/>
+            <origin rpy="0 0 0" xyz="0.25 0 -0.25"/>
             <geometry>
                 <mesh filename="package://tutorial/urdf/head.dae" scale="5 5 5"/>
@@ -10,5 +10,5 @@
         </visual>
         <collision>
-            <origin rpy="0 0 0" xyz="0 0 0"/>
+            <origin rpy="0 0 0" xyz="0.25 0 -0.25"/>
             <geometry>
                 <sphere radius=".2"/>

File: urdf/main.xacro (robot description, xacro)
@@ -5,13 +5,16 @@
     <link name="base_link">
         <visual>
+            <origin rpy="0 0 0" xyz="0 0 0"/>
             <geometry>
-                <box size="1 1 1"/>
+                <box size="1.5 1 0.5"/>
             </geometry>
         </visual>
         <collision>
+            <origin rpy="0 0 0" xyz="0 0 0"/>
             <geometry>
-                <box size="1 1 1"/>
+                <box size="1.5 1 0.5"/>
             </geometry>
         </collision>
+        <origin rpy="0 0 0" xyz="0 0 0"/>
         <inertial>
             <mass value="1"/>
@@ -19,6 +22,8 @@
         </inertial>
     </link>
-    <xacro:arm prefix="right" length=".7" radius=".2" reflect="1" />
-    <xacro:arm prefix="left" length=".7" radius=".2" reflect="-1" />
+    <xacro:arm prefix="front_right" length=".125" radius=".5" reflect_x="1" reflect_y= "1"/>
+    <xacro:arm prefix="front_left" length=".125" radius=".5" reflect_x="1" reflect_y= "-1"/>
+    <xacro:arm prefix="back_right" length=".125" radius=".5" reflect_x="-1" reflect_y="1"/>
+    <xacro:arm prefix = "back_left" length=".125" radius=".5" reflect_x="-1" reflect_y="-1"/>
     <xacro:head />
     <!-- Add ROS plugin so we can interact with our robot -->

Commit message: made a funky looking wheel bot

File: urdf/arm.xacro (robot description, xacro)
@@ -6,5 +6,5 @@
     <link name="${prefix}_arm">
         <visual>
-            <origin rpy="0 0 0" xyz="0 0 1"/> <!-- set the origin to 0 to recenter the link to the child_frame -->
+            <origin rpy="4pi/2 0 0" xyz="0 0.5 0"/> <!-- set the origin to 0 to recenter the link to the child_frame -->
             <geometry>
                 <cylinder length="${length}" radius="${radius}"/>
@@ -12,5 +12,5 @@
         </visual>
         <collision>
-            <origin rpy="0 0 0" xyz="0 0 1"/> <!-- set the origin to 0 to recenter the link to the child_frame -->
+            <origin rpy="4pi/2 0 0" xyz="0 0.5 0"/> <!-- set the origin to 0 to recenter the link to the child_frame -->
             <geometry>
                 <cylinder length="${length}" radius="${radius}"/>
@@ -18,5 +18,5 @@
         </collision>
         <inertial>
-            <origin rpy="0 0 0" xyz="0 0 1"/> <!-- set the origin to 0 to recenter the link to the child_frame -->
+            <origin rpy="4pi/2 0 0" xyz="0 0.5 0"/> <!-- set the origin to 0 to recenter the link to the child_frame -->
             <mass value="1"/>
             <inertia ixx="0.06" ixy="0.0" ixz="0.0" iyy="0.06" iyz="0.0" izz="0.25"/>
@@ -24,8 +24,8 @@
     </link>
     <joint name="base_to_${prefix}_arm" type="continuous">
-        <axis xyz="0 1 0"/>
+        <axis xyz="0 0.5 0"/>
         <parent link="base_link"/>
         <child link="${prefix}_arm"/>
-        <origin rpy="0.2 0 0" xyz="0 ${reflect*0.7} 0"/> <!-- move the child_frame with respect to parent_frame -->
+        <origin rpy="0 0 0" xyz="0 ${reflect*0} 0"/> <!-- move the child_frame with respect to parent_frame -->
         <limit effort="30" velocity="1.0"/>
     </joint>

File: urdf/main.xacro (robot description, xacro)
@@ -6,10 +6,10 @@
         <visual>
             <geometry>
-                <box size="1 1 1"/>
+                <box size="1 1 0.5"/>
             </geometry>
         </visual>
         <collision>
             <geometry>
-                <box size="1 1 1"/>
+                <box size="1 1 0.5"/>
             </geometry>
         </collision>
@@ -19,6 +19,6 @@
         </inertial>
     </link>
-    <xacro:arm prefix="right" length=".7" radius=".2" reflect="1" />
-    <xacro:arm prefix="left" length=".7" radius=".2" reflect="-1" />
+    <xacro:arm prefix="right" length=".1" radius=".5" reflect="1" />
+    <xacro:arm prefix="left" length=".1" radius=".5" reflect="-1" />
     <xacro:head />
     <!-- Add ROS plugin so we can interact with our robot -->
