Commit message: Computer vision

File: urdf/camera.xacro (robot description, xacro)
@@ -1,5 +1,5 @@
 <?xml version="1.0"?>
 <robot xmlns:xacro="http://www.ros.org/wiki/xacro" name="sumo">
-  <xacro:macro name="camera">
+  <xacro:macro name="front_camera" params="name">
     <!-- Camera -->
     <link name="camera_link">

File: urdf/sumo.urdf.xacro (robot description, xacro)
@@ -22,5 +22,5 @@
   <xacro:wheel prefix="right" radius="0.05" reflect="1" />
   <xacro:wheel prefix="left" radius="0.05" reflect="-1" />
-  <xacro:camera />
+  <xacro:front_camera name = "camera" />
   <link name="back_wheel">
     <visual>

Commit message: add new course, rename package

File: urdf/camera.xacro (robot description, xacro)
@@ -6,5 +6,5 @@
       <visual>
         <geometry>
-          <mesh filename="package://sumo/meshes/head.dae" scale=".5 .5 .5"/>
+          <mesh filename="package://computer_vision_pkg/meshes/head.dae" scale=".5 .5 .5"/>
         </geometry>
       </visual>

File: urdf/sumo.urdf.xacro (robot description, xacro)
@@ -1,6 +1,6 @@
 <?xml version="1.0"?>
 <robot xmlns:xacro="http://www.ros.org/wiki/xacro" name="sumo">
-  <xacro:include filename="$(find sumo)/urdf/wheel.xacro" />
-  <xacro:include filename="$(find sumo)/urdf/camera.xacro" />
+  <xacro:include filename="$(find computer_vision_pkg)/urdf/wheel.xacro" />
+  <xacro:include filename="$(find computer_vision_pkg)/urdf/camera.xacro" />
   <xacro:property name="base_length" value=".15" />
   <link name="base_link">
