Commit message: Ready for exercise

File: urdf/sumo.urdf.xacro (robot description, xacro)
@@ -43,5 +43,5 @@
     </collision>
     <inertial>
-      <mass value="0.10"/>
+      <mass value="0.5"/>
       <inertia ixx="0.03" ixy="0.0" ixz="0.0" iyy="0.03" iyz="0.0" izz="0.03"/>
     </inertial>

Commit message: remove friction of backwheel, lower body to prevent robot from rocking

File: urdf/sumo.urdf.xacro (robot description, xacro)
@@ -33,15 +33,7 @@
         <sphere radius="0.02"/>
       </geometry>
-      <surface>
-        <friction>
-          <ode>
-            <mu>200.0</mu>
-            <mu2>100.0</mu2>
-          </ode>
-        </friction>
-      </surface>
     </collision>
     <inertial>
-      <mass value="0.5"/>
+      <mass value="1"/>
       <inertia ixx="0.03" ixy="0.0" ixz="0.0" iyy="0.03" iyz="0.0" izz="0.03"/>
     </inertial>
@@ -50,6 +42,22 @@
     <parent link="base_link"/>
     <child link="back_wheel"/>
-    <origin rpy="0 0 0" xyz="-0.06 0.00 -0.03"/>
+    <origin rpy="0 0 0" xyz="-0.04 0.00 -0.02"/>
   </joint>
+  <gazebo reference="back_wheel">
+    <material>Gazebo/Blue</material>
+    <mu1>0.0</mu1>
+    <mu2>0.0</mu2>
+    <slip1>1.0</slip1>
+    <slip2>1.0</slip2>
+    <selfCollide>true</selfCollide>
+    <gravity>true</gravity>
+  </gazebo>
+  <gazebo reference="base_link">
+    <material>Gazebo/White</material>
+    <mu1>0.0</mu1>
+    <mu2>0.0</mu2>
+    <selfCollide>true</selfCollide>
+    <gravity>true</gravity>
+  </gazebo>
   <!-- Add ROS plugin so we can interact with our robot -->
   <gazebo>

File: urdf/wheel.xacro (robot description, xacro)
@@ -30,5 +30,5 @@
       <parent link="base_link"/>
       <child link="${prefix}_wheel"/>
-      <origin rpy="1.57075 0 0" xyz=".05 ${0.06*reflect} 0.00"/>
+      <origin rpy="1.57075 0 0" xyz=".03 ${0.06*reflect} 0.01"/>
     </joint>
     <transmission name="${prefix}_wheel_transmission">
